File: Power.kicad_sch (KiCad schematic)
At the start: 17 parts, among them J1 USB_C_Receptacle_USB2.0_16P, J2 Conn_Coaxial, U1 STUSB4500QTR, U3 W25Q128JVS, U4 74HC4051, U5 LM2902, U6 TPS55289RYQR, U7 ESP32-C3, Y1 X322540MPB4SI

Commit message: Почти завершённая схема
Parts:
- removed D1: ESDA25P35-1U1M, ESDA25P35-1U1M:ESDA25P351U1M, symbol ESDA25P35-1U1M:ESDA25P35-1U1M
- removed D3: WS2812B, LED_SMD:LED_WS2812B_PLCC4_5.0x5.0mm_P3.2mm, symbol LED:WS2812B
- removed J2: Conn_Coaxial, Connector_Coaxial:U.FL_Hirose_U.FL-R-SMT-1_Vertical, symbol Connector:Conn_Coaxial
- removed U4: 74HC4051, PCM_Package_SO_AKL:TSSOP-16_4.4x5mm_P0.65mm, symbol 74xx:74HC4051
- removed U5: LM2902, PCM_Package_SO_AKL:TSSOP-14_4.4x5mm_P0.65mm, symbol Amplifier_Operational:LM2902
- added AE1: ADWH002, Resistor_SMD:R_1206_3216Metric, symbol Device:Antenna_Chip
- added C10, C11, C4, C9: 1uF, Capacitor_SMD:C_0402_1005Metric, symbol Device:C
- added C12, C13, C14, C17, C18, C19, C20, C21, C22, C23, C24, C25, C28, C29, C30, C32, C34, C45, C46, C5, C53, C54, C6, C7, C8: 22uF, Capacitor_SMD:C_0805_2012Metric, symbol Device:C
- added C15, C31: 10pF, Capacitor_SMD:C_0402_1005Metric, symbol Device:C
- added C16, C33: 2.4nF, Capacitor_SMD:C_0402_1005Metric, symbol Device:C
- added C26, C27, C3, C35, C50, C51, C52, C55, C56, C57, C58, C59, C62: 100nF, Capacitor_SMD:C_0402_1005Metric, symbol Device:C
- added C36, C37, C38, C39, C40, C41, C43, C44: 47uF, Capacitor_SMD:C_0805_2012Metric, symbol Device:C
- added C42: 4.7uF, Capacitor_SMD:C_0402_1005Metric, symbol Device:C
- added C47, C48: 22uF, Capacitor_SMD:C_0402_1005Metric, symbol Device:C
- added C49: 10uF, Capacitor_SMD:C_0402_1005Metric, symbol Device:C
- added C60, C61: 24pF, Capacitor_SMD:C_0201_0603Metric, symbol Device:C
- added C63: 1.8pF, Capacitor_SMD:C_0201_0603Metric, symbol Device:C
- added C64: 1.2pF, Capacitor_SMD:C_0201_0603Metric, symbol Device:C
- added D10, D7, D8, D9: LED, LED_SMD:LED_0402_1005Metric, symbol Device:LED
- added D5: ESDA25P35-1U1M, ESDA25P35-1U1M:ESDA25P351U1M, symbol ESDA25P35-1U1M:ESDA25P35-1U1M
- added D6: SS34, Diode_SMD:D_SMA, symbol PCM_Diode_Schottky_AKL:SS34
- added DA1: TPS7A5701RTER, TPS7A57:TPS7A57, symbol TPS7A5701RTER:TPS7A5701RTER
- added J3: Barrel_Jack_MountingPin, Connector_BarrelJack:BarrelJack_GCT_DCJ200-10-A_Horizontal, symbol Connector:Barrel_Jack_MountingPin
- added L2: IHLP4040DZER4R7M01, Inductor_SMD:L_APV_APH1040, symbol Device:L
- added L3: IHLP4040DZER100M01, Inductor_SMD:L_APV_APH1040, symbol Device:L
- added L4: 24nH, Inductor_SMD:L_0201_0603Metric, symbol Device:L
- added L5: 3nH, Inductor_SMD:L_0201_0603Metric, symbol Device:L
- added Q1, Q2: STL6P3LLH6, STL6P3LLH6:STL8N10F7, symbol STL6P3LLH6:STL6P3LLH6
- added R1, R20, R7, R8: 100K, PCM_Resistor_SMD_AKL:R_0402_1005Metric, symbol Device:R
- added R10, R17: 70.6K, PCM_Resistor_SMD_AKL:R_0402_1005Metric, symbol Device:R
- added R11, R15: 82K, PCM_Resistor_SMD_AKL:R_0402_1005Metric, symbol Device:R
- added R12, R16: 10K, PCM_Resistor_SMD_AKL:R_0402_1005Metric, symbol Device:R
- added R13, R14: 0, PCM_Resistor_SMD_AKL:R_0402_1005Metric, symbol Device:R
- added R18, R22, R23, R9: 0.01, PCM_Resistor_SMD_AKL:R_0402_1005Metric, symbol Device:R
- added R19: 49.9K, PCM_Resistor_SMD_AKL:R_0402_1005Metric, symbol Device:R
- added R2: 22K, PCM_Resistor_SMD_AKL:R_0402_1005Metric, symbol Device:R
- added R21: 16.9K, PCM_Resistor_SMD_AKL:R_0402_1005Metric, symbol Device:R
- added R24: 620, Resistor_SMD:R_0402_1005Metric, symbol Device:R
- added R25: 1.5K, Resistor_SMD:R_0402_1005Metric, symbol Device:R
- added R26, R27: 10K, Resistor_SMD:R_0402_1005Metric, symbol Device:R
- added R28, R29, R30, R31, R32, R33, R36, R37, R38, R39, R40, R41, R45, R46, R47, R48, R50: 0, PCM_Resistor_SMD_AKL:R_0201_0603Metric, symbol Device:R
- added R3: 100, PCM_Resistor_SMD_AKL:R_0402_1005Metric, symbol Device:R
- added R34, R49: 100K, PCM_Resistor_SMD_AKL:R_0201_0603Metric, symbol Device:R
- added R35, R44: 10K, PCM_Resistor_SMD_AKL:R_0201_0603Metric, symbol Device:R
- added R4: 470, PCM_Resistor_SMD_AKL:R_0402_1005Metric, symbol Device:R
- added R42, R43: 4.7K, PCM_Resistor_SMD_AKL:R_0402_1005Metric, symbol Device:R
- added R5, R6: 1K, PCM_Resistor_SMD_AKL:R_0402_1005Metric, symbol Device:R
- added SW1, SW2: TS-1088-AR02016, Button_Switch_SMD:SW_SPST_B3U-1000P, symbol Switch:SW_Push
- added TP1, TP2, TP3, TP4, TP5, TP6: TestPoint, TestPoint:TestPoint_Pad_D1.5mm, symbol Connector:TestPoint
- added TP10, TP11, TP12, TP13, TP14, TP15, TP16, TP7, TP8, TP9: TestPoint, TestPoint:TestPoint_power, symbol Connector:TestPoint
- added U10, U11, U12, U13: INA180A2, Package_TO_SOT_SMD:SOT-23-5, symbol Amplifier_Current:INA180A2
- added U2: LMR16030PDDAR, LMR16030:LMR16030, symbol LMR16030SDDAR:LMR16030PDDAR
- added U5: PCF8575DBR, Package_SO:SSOP-24_5.3x8.2mm_P0.65mm, symbol Interface_Expansion:PCF8575DBR
- added U8: TPS55289RYQR, TPS55289RYQR:TPS55289RYQR, symbol TPS55289RYQR:TPS55289RYQR
- added U9: AP1117-33, Package_TO_SOT_SMD:SOT-223-3_TabPin2, symbol Regulator_Linear:AP1117-33
Connections:
- net at D2.1 (K): now also C4.1, R4.2, R5.1
- net +5V_USB: now reaches D2.2 (A)
- net +5V_USB: now also J1.A4 (VBUS), J1.A9 (VBUS), J1.B4 (VBUS), J1.B9 (VBUS), C5.1, C6.1, C7.1, Q1.5 (D_1), Q1.6 (D_2), Q1.7 (D_3), R26.2, R4.1
- net at D4.1 (L1): now also J1.A5 (CC1), U1.1 (CC1DB), U1.2 (CC1)
- net Earth: now reaches D4.2 (VN)
- net Earth: now also DD1.3 (GND), DD1.7 (L), J1.A1 (GND), J1.A12 (GND), J1.B1 (GND), J1.B12 (GND), J1.S1 (SHIELD), U1.10 (GND), U1.22 (VSYS), U1.25 (GND), U1.3 (NC), U3.4 (GND), U6.17 (AGND), U6.22 (PGND_2), U6.23 (PGND_3), U6.9 (PGND_1), U7.33 (GND), Y1.2, Y1.4, C10.2, C11.2, C12.2, C13.2, C14.2, C15.2, C16.2, C17.2, C18.2, C19.2, C20.2, C21.2, C22.2, C23.2, C24.2, C25.2, C28.2, C29.2, C30.2, C31.2, C32.2, C33.2, C34.2, C36.2, C37.2, C38.2, C39.2, C4.2, C40.2, C41.2, C42.2, C43.2, C44.2, C45.2, C46.2, C47.2, C48.2, C49.2, C5.2, C50.2, C51.2, C52.2, C53.2, C54.2, C55.2, C56.2, C57.2, C58.2, C59.2, C6.2, C60.2, C61.2, C62.2, C63.2, C64.2, C7.2, C8.2, C9.2, D10.1 (K), D5.2 (A), D6.2 (A), D7.1 (K), D8.1 (K), D9.1 (K), DA1.14 (PG), DA1.15 (CP_EN), DA1.17 (EP), DA1.6 (GND), J3.2, R11.2, R12.2, R13.2, R14.2, R15.2, R19.2, R21.2, R7.2, R8.2, SW1.2, SW2.2, TP11.1, TP12.1, TP13.1, TP14.1, TP16.1, U10.2 (GND), U11.2 (GND), U12.2 (GND), U13.2 (GND), U2.7 (GND), U2.9 (EP), U8.17 (AGND), U8.22 (PGND_2), U8.23 (PGND_3), U8.9 (PGND_1), U9.1 (GND)
- net at D4.3 (L2): now also J1.B5 (CC2), U1.4 (CC2), U1.5 (CC2DB)
- net SPICS0: now reaches U3.1 (~{CS})
- net SPICS0: now also R30.2
- net SPIQ: now reaches U3.2 (DO/IO_{1})
- net SPIQ: now also R33.2
- net SPIWP: now reaches U3.3 (~{WP}/IO_{2})
- net SPIWP: now also R29.2
- net SPID: now reaches U3.5 (DI/IO_{0})
- net SPID: now also R32.2
- net SPICLK: now reaches U3.6 (CLK)
- net SPICLK: now also R31.2
- net SPIHD: now reaches U3.7 (~{HOLD})
- net SPIHD: now also R28.2
- net +3.3V_LDO: now reaches U3.8 (VCC)
- net +3.3V_LDO: now also DD1.2 (VDD), C48.1, C49.1, C50.1, C55.1, C56.1, C57.1, C58.1, C59.1, C62.1, R24.2, R34.2, R35.2, R42.1, R43.1, R44.2, R49.2, U10.5 (V+), U11.5 (V+), U12.5 (V+), U13.5 (V+), U9.2 (VO)
- net at U1.12 (ADDR0): now also R8.1
- net at U1.13 (ADDR1): now also R7.1
- net VBUS_EN_SNK: now reaches U1.16 (VBUS_EN_SNK)
- net VBUS_EN_SNK: now also R2.2
- net VBUS_VS_DISH: now reaches U1.18 (VBUS_VS_DISCH)
- net VBUS_VS_DISH: now also R5.2
- net at U1.19 (ALERT): now also TP1.1
- net at U1.21 (VREG_1V2): now also C10.1
- net at U1.23 (VREG_2V7): now also C9.1
- net PD_VDD: now reaches U1.24 (VDD)
- net PD_VDD: now also C11.1, Q1.1 (S_1), Q1.2 (S_2), Q1.3 (S_3), Q2.1 (S_1), Q2.2 (S_2), Q2.3 (S_3), R1.1
- net PD-RST: now reaches U1.6 (RESET)
- net PD-RST: now also U5.6 (P2)
- net SCL: now reaches U1.7 (SCL)
- net SCL: now also U6.3 (SCL), R40.1, R43.2, U8.3 (SCL)
- net SDA: now reaches U1.8 (SDA)
- net SDA: now also U6.4 (SDA), R41.1, R42.2, U8.4 (SDA)
- net DISH: now reaches U1.9 (DISCH)
- net DISH: now also R6.1
- net TPS1_EN: now reaches U6.1 (EN/UVLO)
- net TPS1_EN: now also U5.4 (P0)
- net VOUT1_: now reaches U6.11 (VOUT)
- net VOUT1_: now also U6.12 (ISP), C12.1, C13.1, C14.1, C8.1, R9.1, U10.3 (+)
- net VOUT1: now reaches U6.13 (ISN)
- net VOUT1: now also C17.1, R9.2, TP7.1, U10.4 (-)
- net at U6.14 (FB/~{INT}): now also TP2.1
- net at U6.15 (COMP): now also C15.1, R10.1
- net at U6.16 (CDC): now also TP3.1
- net at U6.18 (VCC): now also U6.21 (EXTVCC), C18.1
- net at U6.2 (MODE): now also R12.1
- net at U6.5 (DITH/SYNC): now also R13.1
- net at U6.6 (FSW): now also R11.1
- net PD-Voltage: now reaches U6.7 (VIN)
- net PD-Voltage: now also C19.1, C20.1, C21.1, C22.1, C23.1, C24.1, C3.1, C45.1, C46.1, C51.1, C52.1, C53.1, C54.1, D5.1 (K), J3.1, Q2.5 (D_1), Q2.6 (D_2), Q2.7 (D_3), R27.2, R6.2, TP15.1, U2.2 (VIN), U2.3 (EN), U8.7 (VIN)
- net at Y1.1: now also U7.29 (XTAL_N), C61.1
- net at Y1.3: now also C60.1, L4.1
- net at U7.1 (LNA_IN): now also C64.1, L5.1
- net GPIO5: now reaches U7.10 (MTDI)
- net GPIO5: now also R47.2
- net GPIO6: now reaches U7.12 (MTCK)
- net GPIO6: now also R45.2
- net GPIO7: now reaches U7.13 (MTDO)
- net GPIO7: now also R46.2
- net GPIO8: now reaches U7.14 (GPIO8)
- net GPIO8: now also R48.2, R49.1
- net GPIO9: now reaches U7.15 (GPIO9)
- net GPIO9: now also R35.1, SW1.1
- net GPIO10: now reaches U7.16 (GPIO10)
- net GPIO10: now also R50.2
- net at U7.19 (SPIHD): now also R28.1
- net at U7.2 (VDD3P3): no longer U7.3 (VDD3P3)
- net at U7.20 (SPIWP): now also R29.1
- net at U7.21 (SPICS0): now also R30.1
- net at U7.22 (SPICLK): now also R31.1
- net at U7.23 (SPID): now also R32.1
- net at U7.24 (SPIQ): now also R33.1
- net GPIO18: now reaches U7.25 (GPIO18)
- net GPIO18: now also R40.2
- net GPIO19: now reaches U7.26 (GPIO19)
- net GPIO19: now also R41.2
- net U0RX: now reaches U7.27 (U0RXD)
- net U0TX: now reaches U7.28 (U0TXD)
- net at U7.30 (XTAL_P): now also L4.2
- net at U7.31 (VDDA): no longer U7.32 (VDDA)
- net GPIO0: now reaches U7.4 (XTAL_32K_P)
- net GPIO0: now also R39.2
- net GPIO1: now reaches U7.5 (XTAL_32K_N)
- net GPIO1: now also R38.2
- net GPIO2: now reaches U7.6 (GPIO2)
- net GPIO2: now also R34.1
- net ESP-EN: now reaches U7.7 (CHIP_EN)
- net ESP-EN: now also R44.1, SW2.1
- net GPIO3: now reaches U7.8 (GPIO3)
- net GPIO3: now also R37.2
- net GPIO4: now reaches U7.9 (MTMS)
- net GPIO4: now also R36.2
- net at DD1.1 (W): now also DA1.7 (REF)
- net SPI_SCLK: now reaches DD1.4 (SCLK)
- net SPI_SCLK: now also R45.1
- net SPI_MOSI: now reaches DD1.5 (DIN)
- net SPI_MOSI: now also R46.1
- net POT_CS: now reaches DD1.6 (~{CS})
- net POT_CS: now also R47.1
- new net: D10.2 (A), R27.1
- new net: AE1.2 (PCB_Trace), C63.1, L5.2
- new net: Q1.4 (G), Q2.4 (G), R1.2, R2.1, R3.1
- new net: D9.2 (A), R26.1
- new net: C25.1, R16.2, U8.18 (VCC), U8.21 (EXTVCC)
- new net: R20.2, R21.1, U2.5 (FB)
- new net: C35.2, D6.1 (K), L3.1, U2.8 (SW)
- new net: C35.1, U2.1 (BOOT)
- new net: C16.1, R10.2
- new net: TP5.1, U8.16 (CDC)
- new net: D7.2 (A), R24.1
- new net: C26.1, L2.1, U8.8 (SW1)
- new net: C26.2, U8.20 (BOOT1)
- new net: C33.1, R17.2
- new net: TP4.1, U8.14 (FB/~{INT})
- new net: R19.1, U2.4 (RT/SYNC)
- new net: TP6.1, U2.6 (PG)
- new net: D8.2 (A), R25.1
- new net: R16.1, U8.2 (MODE)
- new net: R14.1, U8.5 (DITH/SYNC)
- new net: C3.2, R3.2
- new net: C31.1, R17.1, U8.15 (COMP)
- new net: C27.1, L2.2, U8.10 (SW2)
- new net: C27.2, U8.19 (BOOT2)
- new net: C42.1, DA1.8 (NR/SS)
- new net: R15.1, U8.6 (FSW)
- new net +5.2V: C36.1, C37.1, C47.1, DA1.1 (IN_1), DA1.2 (IN_2), DA1.3 (IN_3), DA1.4 (IN_4), DA1.5 (BIAS), R23.2, TP10.1, U13.4 (-), U9.3 (VI)
- new net +5.2V_: C43.1, C44.1, L3.2, R20.1, R23.1, R25.2, U13.3 (+)
- new net CURR_SENSE_1: R39.1, U10.1
- new net CURR_SENSE_2: R38.1, U11.1
- new net CURR_SENSE_3: R37.1, U12.1
- new net CURR_SENSE_4: R36.1, U13.1
- new net LDO_EN: DA1.16 (EN)
- new net ST7789_CS: R48.1
- new net ST7789_DC: R50.1
- new net TPS2_EN: U5.5 (P1), U8.1 (EN/UVLO)
- new net VOUT2: C34.1, R18.2, TP8.1, U11.4 (-), U8.13 (ISN)
- new net VOUT2_: C28.1, C29.1, C30.1, C32.1, R18.1, U11.3 (+), U8.11 (VOUT), U8.12 (ISP)
- new net VOUT3: R22.2, TP9.1, U12.4 (-)
- new net VOUT3_: C38.1, C39.1, C40.1, C41.1, DA1.10 (OUT_2), DA1.11 (OUT_3), DA1.12 (OUT_4), DA1.13 (SNS), DA1.9 (OUT_1), R22.1, U12.3 (+)
- no-connect marks 0 -> 15
Other:
- note added: "1)Подключить выключатели питания для 3х доменов а также общий выключатель без которого бы не было б управления 2)добавить внешние коннекторы для дисплея и кнопок 3)Добавить тестпоинты на I2C и SPI шины 4)Вывести и неиспользуемые пины расширителя пинов 5)Поставить неиспользуемый второй модуль расширения пинов но уже с другим адресом и выводом на тестовые пины - как бы на вырост"
- note added: "12-20V 5A"
- note removed: "Замер тока будет через шунты 0.01 Ом Включение и выключение быдет соответственно по пинам EN ( для всех кроме прямо с БП )"
- moved on the sheet: C1, C2, D2, D4, DD1, J1, L1, U3, U6, Y1
