File: USB-PD-Voltage-supply.kicad_sch (KiCad schematic)
At the start: 16 parts, among them J1 USB_C_Receptacle_USB2.0_16P, J2 Conn_Coaxial, U1 STUSB4500QTR, U3 W25Q128JVS, U4 74HC4051, U5 LM2902, U6 TPS55289RYQR, U7 ESP32-C3, Y1 X322540MPB4SI

Commit message: upd
Parts:
- removed C1, C2: 100nF, Capacitor_SMD:C_0402_1005Metric, symbol Device:C
- removed D1: ESDA25P35-1U1M, ESDA25P35-1U1M:ESDA25P351U1M, symbol ESDA25P35-1U1M:ESDA25P35-1U1M
- removed D2: SS34, Diode_SMD:D_SMA, symbol PCM_Diode_Schottky_AKL:SS34
- removed D3: WS2812B, LED_SMD:LED_WS2812B_PLCC4_5.0x5.0mm_P3.2mm, symbol LED:WS2812B
- removed DD1: TPL0501-100DCNR, TPL0501-100DCNR:SOT65P280X145-8N, symbol TPL0501-100DCNR:TPL0501-100DCNR
- removed J1: USB_C_Receptacle_USB2.0_16P, Connector_USB:USB_C_Receptacle_G-Switch_GT-USB-7010ASV, symbol Connector:USB_C_Receptacle_USB2.0_16P
- removed J2: Conn_Coaxial, Connector_Coaxial:U.FL_Hirose_U.FL-R-SMT-1_Vertical, symbol Connector:Conn_Coaxial
- removed L1: IHLP4040DZER4R7M01, Inductor_SMD:L_APV_APH1040, symbol Device:L
- removed U1: STUSB4500QTR, Package_DFN_QFN:QFN-24-1EP_4x4mm_P0.5mm_EP2.7x2.7mm, symbol Interface_USB:STUSB4500QTR
- removed U3: W25Q128JVS, Package_SO:SOIC-8_5.3x5.3mm_P1.27mm, symbol Memory_Flash:W25Q128JVS
- removed U4: 74HC4051, PCM_Package_SO_AKL:TSSOP-16_4.4x5mm_P0.65mm, symbol 74xx:74HC4051
- removed U5: LM2902, PCM_Package_SO_AKL:TSSOP-14_4.4x5mm_P0.65mm, symbol Amplifier_Operational:LM2902
- removed U6: TPS55289RYQR, TPS55289RYQR:TPS55289RYQR, symbol TPS55289RYQR:TPS55289RYQR
- removed U7: ESP32-C3, Package_DFN_QFN:QFN-32-1EP_5x5mm_P0.5mm_EP3.7x3.7mm, symbol MCU_Espressif:ESP32-C3
- removed Y1: X322540MPB4SI, Crystal:Crystal_SMD_3225-4Pin_3.2x2.5mm, symbol Device:Crystal_GND24_Small
Other:
- added sheet MCU (MCU.kicad_sch)
- added sheet Power (Power.kicad_sch)
- note removed: "Замер тока будет через шунты 0.01 Ом Включение и выключение быдет соответственно по пинам EN ( для всех кроме прямо с БП )"

Commit message: Почти завершённая схема
Other:
- note added: "Curr-amp"
- note added: "INA180"
- note removed: "74HC4051"
- note removed: "8xAnalog switch"
- note removed: "Current sense 5"
- note removed: "LM2902"
- note removed: "OP-Amp"

Commit message: Schematics done
Other:
- sheet Power renamed main
- removed sheet MCU
- sheet main: file Power.kicad_sch -> main.kicad_sch
- note added: "240*320 display"
- note added: "PCA9555"
- note added: "USBx2"
- note added: "Схема электрическая"
- note added: "Узел печатный источник"
- note added: "питания многоканальный"
- note added: "принципиальная"
- note removed: "240*240 display"
- note removed: "PCF8575TS/1"
- note removed: "USB"
